File: design/power_supply.kicad_sch (KiCad schematic)
At the start: 0 parts

Commit message: Commit antes del merge
Parts:
- added C50, C54: 680uF, Capacitor_THT:CP_Radial_D6.3mm_P2.50mm, symbol Device:C_Small
Connections:
- new net GND: C50.2, C54.2
- new net SUPPLY: C50.1, C54.1
