File: design/mcu.kicad_sch (KiCad schematic)
At the start: 13 parts, among them U1 STM32F40X_LQFP64, X1 8MHz

Commit message: Correccion de DRC
Parts:
- U1: LCSC (none) -> C1339473
Changed lines of the file:
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@@
+			)
+		)
+		(property "LCSC" "C1339473"
+			(at 153.67 86.36 0)
+			(effects
+				(font
+					(size 1.27 1.27)
+				)
+				(hide yes)
 			)
 		)

Commit message: Agrego # de los cristales
Parts:
- X1: LCSC (none) -> C259040; MPN ABLS-8.000MHZ-B4-T -> C08000J060; Manufacturer Abracon LLC -> ECEC(ZheJiang E ast Crystal Elec)
Changed lines of the file:
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@@
 			)
 		)
-		(property "Manufacturer" "Abracon LLC"
+		(property "Manufacturer" " ECEC(ZheJiang E ast Crystal Elec)"
 			(at 205.74 39.37 0)
 			(effects
@@
 			)
 		)
-		(property "MPN" "ABLS-8.000MHZ-B4-T"
+		(property "MPN" "C08000J060"
 			(at 205.74 39.37 0)
 			(effects
+				(font
+					(size 1.27 1.27)
+				)
+				(hide yes)
+			)
+		)
+		(property "LCSC" "C259040"
+			(at 205.74 39.37 0)
+			(effects

Commit message: Abaratando costos
Cambios en numeros de jlcpcb, pasados a componentes básicos
Parts:
- X1: LCSC C259040 -> C12674
Changed lines of the file:
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@@
 			)
 		)
-		(property "LCSC" "C259040"
+		(property "LCSC" "C12674"
 			(at 205.74 39.37 0)
 			(effects

Commit message: Cambios
Actualizado footprint de USB, cambio de capacitor de feedback por uno básico, pequeños cambios en la ubicación de los footprints.
Parts:
- C1, C7: MPN CL10C150JB8NNNC -> (none); Manufacturer Samsung Electro-Mechanics -> (none)
- C10, C11, C2, C3, C5, C6, C8, C9: MPN CL10A225KO8NNNC -> (none); Manufacturer Samsung Electro-Mechanics -> (none)
- C4: MPN CC0603KRX7R9BB104 -> (none); Manufacturer YAGEO -> (none)
- U1: MPN STM32F401RCT6TR -> (none); Manufacturer STMicroelectronics -> (none)
- X1: MPN C08000J060 -> (none); Manufacturer ECEC(ZheJiang E ast Crystal Elec) -> (none)
Changed lines of the file:
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@@
-			)
-		)
-		(property "Manufacturer" "Samsung Electro-Mechanics"
-			(at 195.58 34.29 0)
-			(effects
-				(font
-					(size 1.27 1.27)
-				)
-				(hide yes)
-			)
-		)
-		(property "MPN" "CL10C150JB8NNNC"
-			(at 195.58 34.29 0)
-			(effects
-				(font
-					(size 1.27 1.27)
-				)
-				(hide yes)
 			)
 		)
@@
 			)
 		)
-		(property "Manufacturer" "Samsung Electro-Mechanics"
-			(at 215.9 34.29 0)
-			(effects
-				(font
-					(size 1.27 1.27)
-				)
-				(hide yes)
-			)
-		)
-		(property "MPN" "CL10C150JB8NNNC"
-			(at 215.9 34.29 0)
-			(effects
-				(font
-					(size 1.27 1.27)
-				)
-				(hide yes)
-			)
-		)
 		(property "LCSC" "C1644"
 			(at 217.17 31.75 0)
@@
 			)
 		)
-		(property "Manufacturer" "YAGEO"
-			(at 199.39 60.96 0)
-			(effects
-				(font
-					(size 1.27 1.27)
-				)
-				(hide yes)
-			)
-		)
-		(property "MPN" "CC0603KRX7R9BB104"
-			(at 199.39 60.96 0)
-			(effects
-				(font
-					(size 1.27 1.27)
-				)
-				(hide yes)
-			)
-		)
 		(property "LCSC" "C14663"
 			(at 202.311 59.7916 0)
@@
 			)
 		)
-		(property "Manufacturer" "Samsung Electro-Mechanics"
-			(at 201.93 129.54 0)
-			(effects
-				(font
-					(size 1.27 1.27)
-				)
-				(hide yes)
-			)
-		)
-		(property "MPN" "CL10A225KO8NNNC"
-			(at 201.93 129.54 0)
-			(effects
-				(font
-					(size 1.27 1.27)
-				)
-				(hide yes)
-			)
-		)
 		(property "LCSC" "C23630"
 			(at 204.47 127 0)
@@
 			)
 		)
-		(property "Manufacturer" "Samsung Electro-Mechanics"
-			(at 210.82 129.54 0)
-			(effects
-				(font
-					(size 1.27 1.27)
-				)
-				(hide yes)
-			)
-		)
-		(property "MPN" "CL10A225KO8NNNC"
-			(at 210.82 129.54 0)
-			(effects
-				(font
-					(size 1.27 1.27)
-				)
-				(hide yes)
-			)
-		)
 		(property "LCSC" "C23630"
 			(at 213.36 127 0)
@@
 			)
 		)
-		(property "Manufacturer" "Samsung Electro-Mechanics"
-			(at 196.85 139.7 0)
-			(effects
-				(font
-					(size 1.27 1.27)
-				)
-				(hide yes)
-			)
-		)
-		(property "MPN" "CL10A225KO8NNNC"
-			(at 196.85 139.7 0)
-			(effects
-				(font
-					(size 1.27 1.27)
-				)
-				(hide yes)
-			)
-		)
 		(property "LCSC" "C23630"
 			(at 199.39 140.97 0)
@@
 			)
 		)
-		(property "Manufacturer" "Samsung Electro-Mechanics"
-			(at 196.85 146.05 0)
-			(effects
-				(font
-					(size 1.27 1.27)
-				)
-				(hide yes)
-			)
-		)
-		(property "MPN" "CL10A225KO8NNNC"
-			(at 196.85 146.05 0)
-			(effects
-				(font
-					(size 1.27 1.27)
-				)
-				(hide yes)
-			)
-		)
 		(property "LCSC" "C23630"
 			(at 199.39 148.59 0)
@@
 			)
 		)
-		(property "Manufacturer" " STMicroelectronics"
-			(at 153.67 86.36 0)
-			(effects
-				(font
-					(size 1.27 1.27)
-				)
-				(hide yes)
-			)
-		)
-		(property "MPN" "STM32F401RCT6TR"
-			(at 153.67 86.36 0)
-			(effects
-				(font
-					(size 1.27 1.27)
-				)
-				(hide yes)
-			)
-		)
 		(property "LCSC" "C1339473"
 			(at 153.67 86.36 0)
@@
 			)
 		)
-		(property "Manufacturer" "Samsung Electro-Mechanics"
-			(at 250.19 46.99 0)
-			(effects
-				(font
-					(size 1.27 1.27)
-				)
-				(hide yes)
-			)
-		)
-		(property "MPN" "CL10A225KO8NNNC"
-			(at 250.19 46.99 0)
-			(effects
-				(font
-					(size 1.27 1.27)
-				)
-				(hide yes)
-			)
-		)
 		(property "LCSC" "C23630"
 			(at 251.46 44.45 0)
@@
 			)
 		)
-		(property "Manufacturer" "Samsung Electro-Mechanics"
-			(at 257.81 46.99 0)
-			(effects
-				(font
-					(size 1.27 1.27)
-				)
-				(hide yes)
-			)
-		)
-		(property "MPN" "CL10A225KO8NNNC"
-			(at 257.81 46.99 0)
-			(effects
-				(font
-					(size 1.27 1.27)
-				)
-				(hide yes)
-			)
-		)
 		(property "LCSC" "C23630"
 			(at 259.08 44.45 0)
@@
 			)
 		)
-		(property "Manufacturer" "Samsung Electro-Mechanics"
-			(at 264.16 46.99 0)
-			(effects
-				(font
-					(size 1.27 1.27)
-				)
-				(hide yes)
-			)
-		)
-		(property "MPN" "CL10A225KO8NNNC"
-			(at 264.16 46.99 0)
-			(effects
-				(font
-					(size 1.27 1.27)
-				)
-				(hide yes)
-			)
-		)
 		(property "LCSC" "C23630"
 			(at 265.43 44.45 0)
@@
 		)
 		(property "Description" "CAP 2.2u, 16V, 0603"
-			(at 270.51 46.99 0)
-			(effects
-				(font
-					(size 1.27 1.27)
-				)
-				(hide yes)
-			)
-		)
-		(property "Manufacturer" "Samsung Electro-Mechanics"
-			(at 270.51 46.99 0)
-			(effects
-				(font
-					(size 1.27 1.27)
-				)
-				(hide yes)
-			)
-		)
-		(property "MPN" "CL10A225KO8NNNC"
 			(at 270.51 46.99 0)
 			(effects
@@
 			(at 205.74 39.37 0)
 			(effects
-				(font
-					(size 1.27 1.27)
-				)
-				(hide yes)
-			)
-		)
-		(property "Manufacturer" " ECEC(ZheJiang E ast Crystal Elec)"
-			(at 205.74 39.37 0)
-			(effects
-				(font
-					(size 1.27 1.27)
-				)
-				(hide yes)
-			)
-		)
-		(property "MPN" "C08000J060"
-			(at 205.74 39.37 0)
-			(effects
